Commit message: Clean project and keep working Gazebo control and closed-loop models

File: urdf/wheel_leg_robot_gazebo_passive_stl.urdf (robot description, URDF)
Before this commit: robot wheel_leg_robot, 11 links, 10 joints
Joints:
- joint big_arm_1_joint: axis (none) -> 0 1 0; limit (none) -> lower=-2.6 upper=2.6 effort=0.0 velocity=20.0; type fixed -> revolute
- joint big_arm_2_joint: axis (none) -> 0 1 0; limit (none) -> lower=-2.6 upper=2.6 effort=0.0 velocity=20.0; type fixed -> revolute
- joint big_arm_3_joint: axis (none) -> 0 1 0; limit (none) -> lower=-2.6 upper=2.6 effort=0.0 velocity=20.0; type fixed -> revolute
- joint big_arm_4_joint: axis (none) -> 0 1 0; limit (none) -> lower=-2.6 upper=2.6 effort=0.0 velocity=20.0; type fixed -> revolute
- joint knee_1_joint: axis (none) -> 0 1 0; limit (none) -> lower=-2.6 upper=2.6 effort=0.0 velocity=20.0; type fixed -> revolute
- joint knee_2_joint: axis (none) -> 0 1 0; limit (none) -> lower=-2.6 upper=2.6 effort=0.0 velocity=20.0; type fixed -> revolute
- joint knee_3_joint: axis (none) -> 0 1 0; limit (none) -> lower=-2.6 upper=2.6 effort=0.0 velocity=20.0; type fixed -> revolute
- joint knee_4_joint: axis (none) -> 0 1 0; limit (none) -> lower=-2.6 upper=2.6 effort=0.0 velocity=20.0; type fixed -> revolute
